File: schematics/link-template/link-template.kicad_pcb (KiCad board)
At the start: 4 copper layers, 76.2 x 79.4 mm, 6 parts, among them J1 PCIE-036-02-X-D-TH, J2 Conn_02x02_Odd_Even, J3 Conn_02x02_Odd_Even

Commit message: update naming, jlc standards, and add text
Other:
- board text added: "OATS Center ??-Link v? (date) ???@purdue.edu"
Changed lines of the file:
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@@
 			)
 			(layer "F.SilkS")
-			(net 1)
 		)
 		(fp_line
@@
 			)
 			(layer "F.SilkS")
-			(net 1)
 		)
 		(fp_line
@@
 			)
 			(layer "F.SilkS")
-			(net 1)
 		)
 		(fp_circle
@@
 			(fill no)
 			(layer "F.SilkS")
-			(net 1)
 		)
 		(fp_line
@@
 			)
 			(layer "F.CrtYd")
-			(net 1)
 		)
 		(fp_line
@@
 			)
 			(layer "F.CrtYd")
-			(net 1)
 		)
 		(fp_line
@@
 			)
 			(layer "F.CrtYd")
-			(net 1)
 		)
 		(fp_line
@@
 			)
 			(layer "F.CrtYd")
-			(net 1)
 		)
 		(fp_line
@@
 			)
 			(layer "F.Fab")
-			(net 1)
 		)
 		(fp_line
@@
 			)
 			(layer "F.Fab")
-			(net 1)
 		)
 		(fp_line
@@
 			)
 			(layer "F.Fab")
-			(net 1)
 		)
 		(fp_line
@@
 			)
 			(layer "F.Fab")
-			(net 1)
 		)
 		(fp_text user "${REFERENCE}"
@@
 			)
 			(layer "Edge.Cuts")
-			(net 1)
 		)
 		(fp_line
@@
 			)
 			(layer "Edge.Cuts")
-			(net 1)
 		)
 		(fp_line
@@
 			)
 			(layer "Edge.Cuts")
-			(net 1)
 		)
 		(fp_line
@@
 			)
 			(layer "Edge.Cuts")
-			(net 1)
 		)
 		(fp_line
@@
 			)
 			(layer "Edge.Cuts")
-			(net 1)
 		)
 		(fp_line
@@
 			)
 			(layer "Edge.Cuts")
-			(net 1)
 		)
 		(fp_line
@@
 			)
 			(layer "Edge.Cuts")
-			(net 1)
 		)
 		(fp_line
@@
 			)
 			(layer "Edge.Cuts")
-			(net 1)
 		)
 		(fp_line
@@
 			)
 			(layer "Edge.Cuts")
-			(net 1)
 		)
 		(fp_line
@@
 			)
 			(layer "Edge.Cuts")
-			(net 1)
 		)
 		(fp_arc
@@
 			)
 			(layer "Edge.Cuts")
-			(net 1)
 		)
 		(fp_line
@@
 			)
 			(layer "F.CrtYd")
-			(net 1)
 		)
 		(fp_line
@@
 			)
 			(layer "F.CrtYd")
-			(net 1)
 		)
 		(fp_line
@@
 			)
 			(layer "F.CrtYd")
-			(net 1)
 		)
 		(fp_line
@@
 			)
 			(layer "F.CrtYd")
-			(net 1)
 		)
 		(fp_text user "PCB Thickness 1.57 mm"
@@
 			)
 			(layer "F.CrtYd")
-			(net 1)
 		)
 		(fp_line
@@
 			)
 			(layer "F.CrtYd")
-			(net 1)
 		)
 		(fp_line
@@
 			)
 			(layer "F.CrtYd")
-			(net 1)
 		)
 		(fp_line
@@
 			)
 			(layer "F.CrtYd")
-			(net 1)
 		)
 		(fp_line
@@
 			)
 			(layer "F.Fab")
-			(net 1)
 		)
 		(fp_line
@@
 			)
 			(layer "F.Fab")
-			(net 1)
 		)
 		(fp_line
@@
 			)
 			(layer "F.Fab")
-			(net 1)
 		)
 		(fp_line
@@
 			)
 			(layer "F.Fab")
-			(net 1)
 		)
 		(pad "1" smd rect
@@
 			)
 			(layer "F.SilkS")
-			(net 1)
 		)
 		(fp_line
@@
 			)
 			(layer "F.SilkS")
-			(net 1)
 		)
 		(fp_line
@@
 			)
 			(layer "F.SilkS")
-			(net 1)
 		)
 		(fp_circle
@@
 			(fill no)
 			(layer "F.SilkS")
-			(net 1)
 		)
 		(fp_line
@@
 			)
 			(layer "F.CrtYd")
-			(net 1)
 		)
 		(fp_line
@@
 			)
 			(layer "F.CrtYd")
-			(net 1)
 		)
 		(fp_line
@@
 			)
 			(layer "F.CrtYd")
-			(net 1)
 		)
 		(fp_line
@@
 			)
 			(layer "F.CrtYd")
-			(net 1)
 		)
 		(fp_line
@@
 			)
 			(layer "F.Fab")
-			(net 1)
 		)
 		(fp_line
@@
 			)
 			(layer "F.Fab")
-			(net 1)
 		)
 		(fp_line
@@
 			)
 			(layer "F.Fab")
-			(net 1)
 		)
 		(fp_line
@@
 			)
 			(layer "F.Fab")
-			(net 1)
 		)
 		(fp_text user "${REFERENCE}"
@@
 			)
 			(layer "F.CrtYd")
-			(net 1)
 		)
 		(fp_line
@@
 			)
 			(layer "F.CrtYd")
-			(net 1)
 		)
 		(fp_line
@@
 			)
 			(layer "F.CrtYd")
-			(net 1)
 		)
 		(fp_line
@@
 			)
 			(layer "F.CrtYd")
-			(net 1)
 		)
 		(fp_line
@@
 			)
 			(layer "F.Fab")
-			(net 1)
 		)
 		(fp_line
@@
 			)
 			(layer "F.Fab")
-			(net 1)
 		)
 		(fp_line
@@
 			)
 			(layer "F.Fab")
-			(net 1)
 		)
 		(fp_line
@@
 			)
 			(layer "F.Fab")
-			(net 1)
 		)
 		(pad "1" smd rect
@@
 			)
 			(layer "F.CrtYd")
-			(net 1)
 		)
 		(fp_line
@@
 			)
 			(layer "F.CrtYd")
-			(net 1)
 		)
 		(fp_line
@@
 			)
 			(layer "F.CrtYd")
-			(net 1)
 		)
 		(fp_line
@@
 			)
 			(layer "F.CrtYd")
-			(net 1)
 		)
 		(fp_line
@@
 			)
 			(layer "F.Fab")
-			(net 1)
 		)
 		(fp_line
@@
 			)
 			(layer "F.Fab")
-			(net 1)
 		)
 		(fp_line
@@
 			)
 			(layer "F.Fab")
-			(net 1)
 		)
 		(fp_line
@@
 			)
 			(layer "F.Fab")
-			(net 1)
 		)
 		(pad "1" smd rect
@@
 		(layer "Edge.Cuts")
 	)
+	(gr_text "OATS Center\n??-Link v?\n(date)\n???@purdue.edu\n"
+		(at 161.4 64.4 0)
+		(layer "F.Mask")
+		(effects
+			(font
+				(size 0.9525 0.9525)
+				(thickness 0.15875)
+				(bold yes)
+			)
+			(justify left bottom)
+		)
+	)
 	(zone
