File: schematics/tc-link/signal.kicad_sch (KiCad schematic)
At the start: 9 parts, among them U1 AD8495

Commit message: update tc-link board
Parts:
- removed C5: 0.1u, symbol Device:C_Small
- C1, C2, C3, C4: footprint (none) -> Capacitor_SMD:C_0402_1005Metric
- R1, R2, R3: footprint (none) -> Resistor_SMD:R_0402_1005Metric
Changed lines of the file:
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@@
-	)
-	(junction
-		(at 156.21 92.71)
-		(diameter 0)
-		(color 0 0 0 0)
-	)
-	(junction
-		(at 156.21 97.79)
-		(diameter 0)
-		(color 0 0 0 0)
 	)
 	(junction
@@
 	(wire
 		(pts
-			(xy 156.21 92.71) (xy 156.21 97.79)
-		)
-		(stroke
-			(width 0)
-			(type default)
-		)
-	)
-	(wire
-		(pts
 			(xy 144.78 68.58) (xy 144.78 69.85)
 		)
@@
 	(wire
 		(pts
-			(xy 156.21 97.79) (xy 156.21 99.06)
-		)
-		(stroke
-			(width 0)
-			(type default)
-		)
-	)
-	(wire
-		(pts
 			(xy 144.78 76.2) (xy 144.78 74.93)
 		)
@@
 	(wire
 		(pts
-			(xy 161.29 80.01) (xy 166.37 80.01)
-		)
-		(stroke
-			(width 0)
-			(type default)
-		)
-	)
-	(wire
-		(pts
-			(xy 156.21 80.01) (xy 156.21 92.71)
-		)
-		(stroke
-			(width 0)
-			(type default)
-		)
-	)
-	(wire
-		(pts
 			(xy 156.21 55.88) (xy 156.21 64.77)
 		)
@@
 	(wire
 		(pts
-			(xy 161.29 97.79) (xy 156.21 97.79)
-		)
-		(stroke
-			(width 0)
-			(type default)
-		)
-	)
-	(wire
-		(pts
 			(xy 144.78 60.96) (xy 144.78 52.07)
 		)
@@
 	(wire
 		(pts
-			(xy 161.29 92.71) (xy 156.21 92.71)
-		)
-		(stroke
-			(width 0)
-			(type default)
-		)
-	)
-	(wire
-		(pts
 			(xy 144.78 68.58) (xy 148.59 68.58)
 		)
@@
 	(wire
 		(pts
+			(xy 156.21 80.01) (xy 156.21 81.28)
+		)
+		(stroke
+			(width 0)
+			(type default)
+		)
+	)
+	(wire
+		(pts
 			(xy 144.78 85.09) (xy 144.78 83.82)
 		)
@@
 	(wire
 		(pts
-			(xy 166.37 80.01) (xy 166.37 81.28)
+			(xy 161.29 80.01) (xy 161.29 81.28)
 		)
 		(stroke
@@
 			)
 		)
-		(property "Footprint" ""
+		(property "Footprint" "Resistor_SMD:R_0402_1005Metric"
 			(at 124.46 68.58 0)
 			(effects
@@
 			)
 		)
-		(property "Footprint" ""
+		(property "Footprint" "Capacitor_SMD:C_0402_1005Metric"
 			(at 144.78 63.5 0)
 			(effects
@@
 				)
 				(path "/8e86abba-54e7-4e79-af31-15eabcc8dc53/cf0945b2-2b77-4b7a-9180-f6abb82eccbe"
-					(reference "C6")
+					(reference "C5")
 					(unit 1)
 				)
@@
 			)
 		)
-		(property "Footprint" ""
+		(property "Footprint" "Resistor_SMD:R_0402_1005Metric"
 			(at 124.46 76.2 0)
 			(effects
@@
 				(path "/8e86abba-54e7-4e79-af31-15eabcc8dc53/cf0945b2-2b77-4b7a-9180-f6abb82eccbe"
 					(reference "R6")
-					(unit 1)
-				)
-			)
-		)
-	)
-	(symbol
-		(lib_id "Device:C_Small")
-		(at 161.29 95.25 0)
-		(unit 1)
-		(exclude_from_sim no)
-		(in_bom yes)
-		(on_board yes)
-		(dnp no)
-		(property "Reference" "C5"
-			(at 163.83 93.726 0)
-			(effects
-				(font
-					(size 1.27 1.27)
-				)
-				(justify left)
-			)
-		)
-		(property "Value" "0.1u"
-			(at 163.83 96.52 0)
-			(effects
-				(font
-					(size 1.27 1.27)
-				)
-				(justify left)
-			)
-		)
-		(property "Footprint" ""
-			(at 161.29 95.25 0)
-			(effects
-				(font
-					(size 1.27 1.27)
-				)
-				(hide yes)
-			)
-		)
-		(property "Datasheet" "~"
-			(at 161.29 95.25 0)
-			(effects
-				(font
-					(size 1.27 1.27)
-				)
-				(hide yes)
-			)
-		)
-		(property "Description" "Unpolarized capacitor, small symbol"
-			(at 161.29 95.25 0)
-			(effects
-				(font
-					(size 1.27 1.27)
-				)
-				(hide yes)
-			)
-		)
-		(pin "2"
-		)
-		(pin "1"
-		)
-		(instances
-			(project ""
-				(path "/8e86abba-54e7-4e79-af31-15eabcc8dc53/185e9162-a4b5-4726-9859-051bc197beb3"
-					(reference "C5")
-					(unit 1)
-				)
-				(path "/8e86abba-54e7-4e79-af31-15eabcc8dc53/cf0945b2-2b77-4b7a-9180-f6abb82eccbe"
-					(reference "C10")
 					(unit 1)
 				)
@@
 	(symbol
 		(lib_id "power:GND")
-		(at 156.21 99.06 0)
+		(at 156.21 81.28 0)
 		(unit 1)
 		(exclude_from_sim no)
@@
 		(on_board yes)
 		(dnp no)
-		(fields_autoplaced yes)
 		(property "Reference" "#PWR09"
-			(at 156.21 105.41 0)
+			(at 156.21 87.63 0)
 			(effects
 				(font
@@
 		)
 		(property "Value" "GND"
-			(at 156.21 104.14 0)
+			(at 156.21 85.09 0)
 			(effects
 				(font
@@
 		)
 		(property "Footprint" ""
-			(at 156.21 99.06 0)
+			(at 156.21 81.28 0)
 			(effects
 				(font
@@
 		)
 		(property "Datasheet" ""
-			(at 156.21 99.06 0)
+			(at 156.21 81.28 0)
 			(effects
 				(font
@@
 		)
 		(property "Description" "Power symbol creates a global label with name \"GND\" , ground"
-			(at 156.21 99.06 0)
+			(at 156.21 81.28 0)
 			(effects
 				(font
@@
 			)
 		)
-		(property "Footprint" ""
+		(property "Footprint" "Capacitor_SMD:C_0402_1005Metric"
 			(at 144.78 72.39 0)
 			(effects
@@
 				)
 				(path "/8e86abba-54e7-4e79-af31-15eabcc8dc53/cf0945b2-2b77-4b7a-9180-f6abb82eccbe"
-					(reference "C7")
+					(reference "C6")
 					(unit 1)
 				)
@@
 			)
 		)
-		(property "Footprint" ""
+		(property "Footprint" "Capacitor_SMD:C_0402_1005Metric"
 			(at 161.29 58.42 0)
 			(effects
@@
 				)
 				(path "/8e86abba-54e7-4e79-af31-15eabcc8dc53/cf0945b2-2b77-4b7a-9180-f6abb82eccbe"
-					(reference "C9")
+					(reference "C8")
 					(unit 1)
 				)
@@
 			)
 		)
-		(property "Footprint" ""
+		(property "Footprint" "Resistor_SMD:R_0402_1005Metric"
 			(at 114.3 82.55 0)
 			(effects
@@
 	(symbol
 		(lib_id "power:GND")
-		(at 166.37 81.28 0)
+		(at 161.29 81.28 0)
 		(unit 1)
 		(exclude_from_sim no)
@@
 		(dnp no)
 		(property "Reference" "#PWR011"
-			(at 166.37 87.63 0)
+			(at 161.29 87.63 0)
 			(effects
 				(font
@@
 		)
 		(property "Value" "GND"
-			(at 166.37 85.344 0)
+			(at 161.29 85.09 0)
 			(effects
 				(font
@@
 		)
 		(property "Footprint" ""
-			(at 166.37 81.28 0)
+			(at 161.29 81.28 0)
 			(effects
 				(font
@@
 		)
 		(property "Datasheet" ""
-			(at 166.37 81.28 0)
+			(at 161.29 81.28 0)
 			(effects
 				(font
@@
 		)
 		(property "Description" "Power symbol creates a global label with name \"GND\" , ground"
-			(at 166.37 81.28 0)
+			(at 161.29 81.28 0)
 			(effects
 				(font
@@
 			)
 		)
-		(property "Footprint" ""
+		(property "Footprint" "Capacitor_SMD:C_0402_1005Metric"
 			(at 144.78 81.28 0)
 			(effects
@@
 				)
 				(path "/8e86abba-54e7-4e79-af31-15eabcc8dc53/cf0945b2-2b77-4b7a-9180-f6abb82eccbe"
-					(reference "C8")
-					(unit 1)
-				)
+					(reference "C7")
+					(unit 1)
+				)
