File: schematics/v1/sim_test/sim_test.kicad_sch (KiCad schematic)
At the start: 13 parts, among them U1 INA849D, U2 OPA182

Commit message: start v2
Parts:
- removed C1, C2: 10nF, Capacitor_SMD:C_0603_1608Metric, symbol Device:C_Small
- removed R5, R6, R9: 1k, Resistor_SMD:R_0603_1608Metric, symbol Device:R_Small_US
- removed R7: 10k, Resistor_SMD:R_0603_1608Metric, symbol Device:R_Small_US
- removed R8: 2k, Resistor_SMD:R_0603_1608Metric, symbol Device:R_Small_US
- removed U2: OPA182, Package_TO_SOT_SMD:SOT-353_SC-70-5, symbol Amplifier_Operational:TLV172IDCK
- removed V3: 3.3, symbol Simulation_SPICE:VDC
- removed V4: VSIN, symbol Simulation_SPICE:VSIN
- removed V5: -3.3, symbol Simulation_SPICE:VDC
- added C8: 5.45n, Capacitor_SMD:C_0402_1005Metric, symbol Device:C_Small
- added C9: 2.72n, Capacitor_SMD:C_0402_1005Metric, symbol Device:C_Small
- added R1: 121, symbol Device:R_Small_US
- added R2, R3: 3.3k, Resistor_SMD:R_0603_1608Metric, symbol Device:R_Small_US
- added R4: 100M, Resistor_SMD:R_0603_1608Metric, symbol Device:R_Small_US
- added U2: OPA1612AxD, Link_Footprints:OPA1612, symbol Amplifier_Operational:OPA1612AxD
- added V2: -12, symbol Simulation_SPICE:VDC
- added V3: VSIN, symbol Simulation_SPICE:VSIN
Connections:
- net +12V: now also U2.8 (V+)
- net 0: now also C9.2, R4.1, U2.5 (+), V2.2
- net V_{out}: now reaches U1.7
- net V_{out}: now also R2.1
- net V_{in-}: now reaches U1.1 (-)
- net V_{in-}: now also V3.1
- net at U1.2 (Rg): now also R1.1
- net at U1.3 (Rg): now also R1.2
- net V_{in+}: now reaches U1.4 (+)
- net V_{in+}: now also V3.2
- net -3V3 renamed -12V
- net -12V: now also U2.4 (V-), V2.1
- new net: C8.1, R2.2, R3.1
- new net: U2.6 (-), U2.7
- new net Vf: C8.2, R4.2, U2.1, U2.2 (-)
- new net vp: C9.1, R3.2, U2.3 (+)
- no-connect marks 2 -> 0
Other:
- moved on the sheet: U1, V1
