File: schematics/sim_test/sim_test.kicad_sch (KiCad schematic)
At the start: 13 parts, among them U1 INA849D, U2 OPA182

Commit message: feat(signals): simulates attenuation circuit
Connections:
- net S1- is gone; now on net 0: R5.1, V4.1
Changed lines of the file:
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@@
+	)
+	(junction
+		(at 85.09 43.18)
+		(diameter 0)
+		(color 0 0 0 0)
 	)
 	(junction
@@
 	)
 	(symbol
+		(lib_id "power:GND")
+		(at 85.09 43.18 180)
+		(unit 1)
+		(exclude_from_sim no)
+		(in_bom yes)
+		(on_board yes)
+		(dnp no)
+		(property "Reference" "#PWR019"
+			(at 85.09 36.83 0)
+			(effects
+				(font
+					(size 1.27 1.27)
+				)
+				(hide yes)
+			)
+		)
+		(property "Value" "GND"
+			(at 85.09 39.116 0)
+			(effects
+				(font
+					(size 1.27 1.27)
+				)
+			)
+		)
+		(property "Footprint" ""
+			(at 85.09 43.18 0)
+			(effects
+				(font
+					(size 1.27 1.27)
+				)
+				(hide yes)
+			)
+		)
+		(property "Datasheet" ""
+			(at 85.09 43.18 0)
+			(effects
+				(font
+					(size 1.27 1.27)
+				)
+				(hide yes)
+			)
+		)
+		(property "Description" "Power symbol creates a global label with name \"GND\" , ground"
+			(at 85.09 43.18 0)
+			(effects
+				(font
+					(size 1.27 1.27)
+				)
+				(hide yes)
+			)
+		)
+		(pin "1"
+		)
+		(instances
+			(project "sim_test"
+				(path "/6ef471a5-3888-443c-aacb-76e5b23708bb"
+					(reference "#PWR019")
+					(unit 1)
+				)
+			)
+		)
+	)
+	(symbol
 		(lib_id "power:-12V")
 		(at 66.04 78.74 0)
@@
 			)
 		)
-		(property "Sim.Params" "dc=0 ampl=1 f=500 ac=10m"
-			(at 47.752 48.26 0)
-			(effects
-				(font
+		(property "Sim.Params" "dc=-1 ampl=1 f=500 ac=1"
+			(at 54.864 48.26 0)
+			(effects
+				(font
