File: schematics/signals/signals.kicad_pcb (KiCad board)
At the start: 4 copper layers, 31.8 x 25.4 mm, 30 parts, among them J1 Conditioned, J2 Sensors, U1 INA849D, U2 OPA2182, U3 INA849D

Commit message: fix(dimensions)
Parts:
- moved J1 0.05 mm to (205.8, 49.4)
Changed lines of the file:
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@@
 		(tags "test point SMD pad")
 		(property "Reference" "TP1"
-			(at 0 -1.448 0)
+			(at -0.635 -1.524 0)
 			(layer "F.SilkS")
 			(effects
@@
 	(footprint "Connector_PinHeader_2.54mm:PinHeader_1x06_P2.54mm_Vertical"
 		(layer "B.Cu")
-		(at 205.7654 49.4538 180)
+		(at 205.7654 49.403 180)
 		(descr "Through hole straight pin header, 1x06, 2.54mm pitch, single row")
 		(tags "Through hole pin header THT 1x06 2.54mm single row")
@@
 	)
 	(gr_text "Signals v1.0"
-		(at 197.866 45.593 0)
+		(at 198.247 45.466 0)
 		(layer "F.Mask")
 		(effects
@@
 		)
 	)
+	(dimension
+		(type orthogonal)
+		(layer "Edge.Cuts")
+		(pts
+			(xy 205.7654 49.403) (xy 205.7654 43.053)
+		)
+		(height 6.0706)
+		(orientation 1)
+		(format
+			(prefix "")
+			(suffix "")
+			(units 3)
+			(units_format 0)
+			(precision 4)
+			(suppress_zeroes yes)
+		)
+		(style
+			(thickness 0.05)
+			(arrow_length 1.27)
+			(text_position_mode 0)
+			(arrow_direction outward)
+			(extension_height 0.58642)
+			(extension_offset 0.5)
+			(keep_text_aligned yes)
+		)
+		(gr_text "0.25"
+			(at 210.686 46.228 90)
+			(layer "Edge.Cuts")
+			(effects
+				(font
+					(size 1 1)
+					(thickness 0.15)
+				)
+			)
+		)
+	)
