File: schematics/link/controller.kicad_sch (KiCad schematic)
At the start: 58 parts, among them J6 Prog_Header, J9 I2C, SW5 nRST, U12 MAX31856, U7 ADS131M02IPWR, U8 STM32G0B1KETx, U9 W5500, Y1 ECS-2520MVLC-081.92-BN-TR, Y2 KC2520Z25.0000C1SY00;

Commit message: GPT review pt2
Parts:
- C27, C29, C31, C33, C35, C36, C37, C38, C39, C40, C41, C42, C43, C44, C52, C54, C55: MPN GRM155R71H104KE14D -> GCM155R71H104KE02D
- C34: value 10uF/16V -> 10uF; MPN GCM21BR71A106KE22L -> GRM21BR61E106MA73L
- R30: footprint Resistor_SMD:R_0603_1608Metric -> Resistor_SMD:R_0402_1005Metric; MPN RT0603BRD07100RL -> RT0402BRD07100RL
Changed lines of the file:
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@@
 			)
 		)
-		(property "MPN" "GRM155R71H104KE14D"
+		(property "MPN" "GCM155R71H104KE02D"
 			(at 101.6 29.21 0)
 			(hide yes)
@@
 			)
 		)
-		(property "MPN" "GRM155R71H104KE14D"
+		(property "MPN" "GCM155R71H104KE02D"
 			(at 74.93 52.07 90)
 			(hide yes)
@@
 			)
 		)
-		(property "MPN" "GRM155R71H104KE14D"
+		(property "MPN" "GCM155R71H104KE02D"
 			(at 196.85 135.89 0)
 			(hide yes)
@@
 			)
 		)
-		(property "MPN" "GRM155R71H104KE14D"
+		(property "MPN" "GCM155R71H104KE02D"
 			(at 228.6 137.16 0)
 			(hide yes)
@@
 			)
 		)
-		(property "MPN" "GRM155R71H104KE14D"
+		(property "MPN" "GCM155R71H104KE02D"
 			(at 83.82 36.83 0)
 			(hide yes)
@@
 			)
 		)
-		(property "MPN" "GRM155R71H104KE14D"
+		(property "MPN" "GCM155R71H104KE02D"
 			(at 34.29 151.13 0)
 			(hide yes)
@@
 			)
 		)
-		(property "MPN" "GRM155R71H104KE14D"
+		(property "MPN" "GCM155R71H104KE02D"
 			(at 113.03 99.06 0)
 			(hide yes)
@@
 			)
 		)
-		(property "MPN" "GRM155R71H104KE14D"
+		(property "MPN" "GCM155R71H104KE02D"
 			(at 63.5 99.06 0)
 			(hide yes)
@@
 			)
 		)
-		(property "MPN" "GRM155R71H104KE14D"
+		(property "MPN" "GCM155R71H104KE02D"
 			(at 50.8 99.06 0)
 			(hide yes)
@@
 			)
 		)
-		(property "Footprint" "Resistor_SMD:R_0603_1608Metric"
+		(property "Footprint" "Resistor_SMD:R_0402_1005Metric"
 			(at 187.96 43.18 0)
 			(hide yes)
@@
 			)
 		)
-		(property "MPN" "RT0603BRD07100RL"
+		(property "MPN" "RT0402BRD07100RL"
 			(at 187.96 43.18 0)
 			(hide yes)
@@
 			)
 		)
-		(property "MPN" "GRM155R71H104KE14D"
+		(property "MPN" "GCM155R71H104KE02D"
 			(at 142.24 83.82 0)
 			(hide yes)
@@
 			)
 		)
-		(property "MPN" "GRM155R71H104KE14D"
+		(property "MPN" "GCM155R71H104KE02D"
 			(at 76.2 99.06 0)
 			(hide yes)
@@
 			)
 		)
-		(property "MPN" "GRM155R71H104KE14D"
+		(property "MPN" "GCM155R71H104KE02D"
 			(at 185.42 135.89 0)
 			(hide yes)
@@
 			)
 		)
-		(property "MPN" "GRM155R71H104KE14D"
+		(property "MPN" "GCM155R71H104KE02D"
 			(at 88.9 99.06 0)
 			(hide yes)
@@
 			)
 		)
-		(property "MPN" "GRM155R71H104KE14D"
+		(property "MPN" "GCM155R71H104KE02D"
 			(at 262.89 38.1 0)
 			(hide yes)
@@
 			)
 		)
-		(property "MPN" "GRM155R71H104KE14D"
+		(property "MPN" "GCM155R71H104KE02D"
 			(at 101.6 99.06 0)
 			(hide yes)
@@
 			)
 		)
-		(property "MPN" "GRM155R71H104KE14D"
+		(property "MPN" "GCM155R71H104KE02D"
 			(at 30.48 99.06 0)
 			(hide yes)
@@
 			)
 		)
-		(property "MPN" "GRM155R71H104KE14D"
+		(property "MPN" "GCM155R71H104KE02D"
 			(at 21.59 168.91 0)
 			(hide yes)
@@
 			)
 		)
-		(property "Value" "10uF/16V"
+		(property "Value" "10uF"
 			(at 20.32 100.3362 0)
 			(show_name no)
@@
 			)
 		)
-		(property "MPN" "GCM21BR71A106KE22L"
+		(property "MPN" "GRM21BR61E106MA73L"
 			(at 17.78 99.06 0)
 			(hide yes)
